File: SmartCube.kicad_pcb (KiCad board)
At the start: 2 copper layers, 3 parts, among them J1 TYPE-C-31-M-12, U1 ESP32-S3-WROOM-1-N8R8, U2 CP2102

Commit message: Add first version of pcb
Parts:
- added BT1: Battery_Cell, Vibrator Motor:vibrator connector, B.Cu at (136.2, 75.3)
- added C1: 22uF, Capacitor_SMD:C_0805_2012Metric, B.Cu at (146.2, 47.9)
- added C10: 10uF, Capacitor_SMD:C_0805_2012Metric, B.Cu at (137.0, 55.0)
- added C11: 10uF, Capacitor_SMD:C_0805_2012Metric, B.Cu at (137.0, 53.0)
- added C12: 1nF, Capacitor_SMD:C_0805_2012Metric, B.Cu at (136.9, 49.0)
- added C13: 22uF, Capacitor_SMD:C_0805_2012Metric, B.Cu at (101.0, 9.40)
- added C14: 22uF, Capacitor_SMD:C_0805_2012Metric, B.Cu at (104.5, 9.40)
- added C15: 0.1uF, Capacitor_SMD:C_0805_2012Metric, B.Cu at (121.2, 15.6)
- added C16: 0.1uF, Capacitor_SMD:C_0805_2012Metric, B.Cu at (59.0, 61.8)
- added C17: 100nF, Capacitor_SMD:C_0805_2012Metric, B.Cu at (56.8, 19.9)
- added C18: 0.1uF, Capacitor_SMD:C_0805_2012Metric, B.Cu at (49.8, 11.8)
- added C19: 0.1uF, Capacitor_SMD:C_0805_2012Metric, B.Cu at (49.8, 19.1)
- added C2: 22uF, Capacitor_SMD:C_0805_2012Metric, B.Cu at (146.2, 49.9)
- added C20: 2.2nF, Capacitor_SMD:C_0805_2012Metric, B.Cu at (53.5, 14.5)
- added C21: 10nF, Capacitor_SMD:C_0805_2012Metric, B.Cu at (45.5, 17.2)
- added C22: 0.1uF, Capacitor_SMD:C_0805_2012Metric, B.Cu at (25.3, 15.6)
- added C23: 104, Capacitor_SMD:C_0805_2012Metric, B.Cu at (145.6, 17.6)
- added C24: 1uF, Capacitor_SMD:C_0805_2012Metric, B.Cu at (123.2, 15.6)
- added C25: 0.1uF, Capacitor_SMD:C_0805_2012Metric, B.Cu at (125.2, 15.6)
- added C29: 22uF, Capacitor_Tantalum_SMD:CP_EIA-3528-21_Kemet-B, B.Cu at (93.1, 7.40)
- added C3: 22uF, Capacitor_SMD:C_0805_2012Metric, B.Cu at (146.2, 51.9)
- added C30: 0.1uF, Capacitor_SMD:C_0805_2012Metric, B.Cu at (92.8, 10.2)
- added C31: 1uF, Capacitor_SMD:C_0805_2012Metric, B.Cu at (92.8, 12.2)
- added C4: 22uF, Capacitor_SMD:C_0805_2012Metric, B.Cu at (146.2, 53.9)
- added C8: 22uF, Capacitor_SMD:C_0805_2012Metric, B.Cu at (132.9, 57.6)
- added C9: 1uF, Capacitor_SMD:C_0805_2012Metric, B.Cu at (132.1, 44.7)
- added D1: LED, LED_SMD:LED_0603_1608Metric, B.Cu at (148.2, 68.5)
- added D10: SP0502BAHT, Package_TO_SOT_SMD:SOT-23, B.Cu at (148.1, 24.7)
- added D11: SP0502BAHT, Package_TO_SOT_SMD:SOT-23, B.Cu at (144.6, 24.8)
- added D2: LED, LED_SMD:LED_0603_1608Metric, B.Cu at (148.3, 70.2)
- added D3: LED, LED_SMD:LED_0603_1608Metric, B.Cu at (148.2, 71.8)
- added D4: LED, LED_SMD:LED_0603_1608Metric, B.Cu at (148.2, 73.3)
- added D5: BZX84Cxx, Package_TO_SOT_SMD:SOT-23, B.Cu at (138.4, 34.5)
- added D7: SS14, Diode_SMD:D_SMA, B.Cu at (22.3, 19.9)
- added D8: WS2812B-4020, WS2812B-4020:LED_WS2812B-4020, B.Cu at (148.8, 16.9)
- added D9: SS14, Diode_SMD:D_SMA, B.Cu at (38.1, 19.6)
- added IP5310: ~, IP5310:IP5310, B.Cu at (137.2, 62.3)
- added J2: XH, Vibrator Motor:vibrator connector, B.Cu at (20.8, 25.9)
- added L1: 1uH, Inductor_SMD:L_7.3x7.3_H4.5, B.Cu at (145.1, 62.8)
- added Q1: AO3401A, Package_TO_SOT_SMD:SOT-23, B.Cu at (138.4, 41.4)
- added Q2: AO3401A, Package_TO_SOT_SMD:SOT-23, B.Cu at (138.4, 44.8)
- added Q3: BC857, Package_TO_SOT_SMD:SOT-23, B.Cu at (138.4, 38.0)
- added Q4: SS8050, Package_TO_SOT_SMD:SOT-23, B.Cu at (113.3, 9.31)
- added Q5: SS8050, Package_TO_SOT_SMD:SOT-23, B.Cu at (116.8, 9.31)
- added Q6: AO3400A, Package_TO_SOT_SMD:SOT-23, B.Cu at (29.2, 23.7)
- added Q7: AO3400A, Package_TO_SOT_SMD:SOT-23, B.Cu at (32.7, 23.7)
- added R1: RSET resistance, Resistor_SMD:R_0805_2012Metric, B.Cu at (135.2, 69.0)
- added R10: 100K, Resistor_SMD:R_0805_2012Metric, B.Cu at (134.1, 41.3)
- added R11: 10K, Resistor_SMD:R_0805_2012Metric, B.Cu at (132.2, 37.9)
- added R12: 1K, Resistor_SMD:R_0805_2012Metric, B.Cu at (134.1, 37.9)
- added R13: 4.7K, Resistor_SMD:R_0805_2012Metric, B.Cu at (119.2, 15.5)
- added R14: 10K, Resistor_SMD:R_0805_2012Metric, B.Cu at (115.3, 15.5)
- added R15: 10K, Resistor_SMD:R_0805_2012Metric, B.Cu at (117.2, 15.5)
- added R16: 10K, Resistor_SMD:R_0805_2012Metric, B.Cu at (59.1, 58.3)
- added R17: 10K, Resistor_SMD:R_0805_2012Metric, B.Cu at (48.5, 58.0)
- added R18: 6, Resistor_SMD:R_0805_2012Metric, B.Cu at (48.5, 61.4)
- added R2: 51K, Resistor_SMD:R_0603_1608Metric, B.Cu at (132.1, 61.6)
- added R23: 10K, Resistor_SMD:R_0805_2012Metric, B.Cu at (35.9, 15.8)
- added R25: 4.7K, Resistor_SMD:R_0805_2012Metric, B.Cu at (92.9, 16.4)
- added R26: R_Shunt, Resistor_SMD:R_Shunt_Vishay_WSK2512_6332Metric_T1.19mm, B.Cu at (30.3, 19.7)
- added R27: 220, Resistor_SMD:R_0805_2012Metric, B.Cu at (37.1, 25.1)
- added R28: 220, Resistor_SMD:R_0805_2012Metric, B.Cu at (37.1, 23.2)
- added R29: 4.7K, Resistor_SMD:R_0805_2012Metric, B.Cu at (92.9, 18.4)
- added R3: OR/NC, Resistor_SMD:R_0805_2012Metric, B.Cu at (139.2, 69.0)
- added R30: 10K, Resistor_SMD:R_0805_2012Metric, B.Cu at (92.9, 14.2)
- added R4: OR/NC, Resistor_SMD:R_0805_2012Metric, B.Cu at (137.2, 69.0)
- added R5: 10K/NC, Resistor_SMD:R_0805_2012Metric, B.Cu at (133.3, 69.0)
- added R6: 10K, Resistor_SMD:R_0805_2012Metric, B.Cu at (134.1, 44.7)
- added R7: 2R, Resistor_SMD:R_0805_2012Metric, B.Cu at (137.0, 51.0)
- added R9: 10K, Resistor_SMD:R_0805_2012Metric, B.Cu at (132.2, 41.3)
- added SW1: SW_Push, Button_Switch_SMD:SW_SPST_EVQP2_MiddlePushTravel_H2.5mm, B.Cu at (147.8, 42.2)
- added U3: SHTC3, Sensor_Humidity:Sensirion_DFN-4-1EP_2x2mm_P1mm_EP0.7x1.6mm, B.Cu at (59.1, 19.8)
- added U4: MPU-6050, Sensor_Motion:InvenSense_QFN-24_4x4mm_P0.5mm, B.Cu at (49.8, 15.4)
- added U5: INA226, Package_SO:VSSOP-10_3x3mm_P0.5mm, B.Cu at (30.5, 15.6)
- added U7: FCC connector, FCC 18 pin 0.5:FPC_18 0.5, B.Cu at (51.6, 55.9)
- added U8: ESP32-S3-WROOM-1, PCM_Espressif:ESP32-S3-WROOM-1, B.Cu at (78.5, 16.7)
- added VibratorMotor1: ~, Vibrator Motor:vibrator connector, B.Cu at (48.0, 25.9)
- added touch_slider2: ~, Touch Slider:TouchSlider-5_50x10mm, F.Cu at (122.7, 52.8)
- J1: value TYPE-C-31-M-12 -> USB_C_Receptacle_USB2.0_16P; footprint TYPE-C-31-M-12:HRO_TYPE-C-31-M-12 -> Connector_USB:USB_C_Receptacle_GCT_USB4105-xx-A_16P_TopMnt_Horizontal; moved to B.Cu
- U1: value ESP32-S3-WROOM-1-N8R8 -> AMS1117-3.3; footprint ESP32-S3-WROOM-1-N8R8:XCVR_ESP32S3WROOM1N8R8 -> Package_TO_SOT_SMD:SOT-223-3_TabPin2; moved to B.Cu
- U2: moved to B.Cu
- moved J1 144.3 mm to (147.4, 32.7), turned to -90 degrees
- moved U1 50.3 mm to (102.8, 15.0), turned to -90 degrees
- moved U2 46.4 mm to (123.1, 9.35), turned to 90 degrees
Connections:
- J1 pad A5: unconnected-(J1-CC1-PadA5) -> /CC1
- J1 pad A6: unconnected-(J1-DP1-PadA6) -> /D+
- J1 pad A7: unconnected-(J1-DN1-PadA7) -> /D-
- J1 pad B5: unconnected-(J1-CC2-PadB5) -> /CC2
- J1 pad B6: unconnected-(J1-DP2-PadB6) -> /D+
- J1 pad B7: unconnected-(J1-DN2-PadB7) -> /D-
- J1 pad S1: Net-(J1-SHIELD-PadS1) -> GND
- U1 pad 1: Net-(U1-GND-Pad1) -> GND
- U1 pad 2: unconnected-(U1-3V3-Pad2) -> /V3.3
- U1 pad 3: unconnected-(U1-EN-Pad3) -> /VOUT
- U2 pad 10: Net-(U2-NC-Pad10) -> unconnected-(U2-NC-Pad10)_6
- U2 pad 13: Net-(U2-NC-Pad10) -> unconnected-(U2-NC-Pad10)_8
- U2 pad 14: Net-(U2-NC-Pad10) -> unconnected-(U2-NC-Pad10)_7
- U2 pad 15: Net-(U2-NC-Pad10) -> unconnected-(U2-NC-Pad10)_5
- U2 pad 16: Net-(U2-NC-Pad10) -> unconnected-(U2-NC-Pad10)
- U2 pad 17: Net-(U2-NC-Pad10) -> unconnected-(U2-NC-Pad10)_4
- U2 pad 18: Net-(U2-NC-Pad10) -> unconnected-(U2-NC-Pad10)_1
- U2 pad 19: Net-(U2-NC-Pad10) -> unconnected-(U2-NC-Pad10)_2
- U2 pad 20: Net-(U2-NC-Pad10) -> unconnected-(U2-NC-Pad10)_3
- U2 pad 21: Net-(U2-NC-Pad10) -> unconnected-(U2-NC-Pad10)_9
- U2 pad 22: Net-(U2-NC-Pad10) -> unconnected-(U2-NC-Pad10)_10
- U2 pad 24: unconnected-(U2-RTS-Pad24) -> /RTS
- U2 pad 25: unconnected-(U2-RXD-Pad25) -> /TX0
- U2 pad 26: unconnected-(U2-TXD-Pad26) -> /RX0
- U2 pad 28: unconnected-(U2-DTR-Pad28) -> /DTR
- U2 pad 29: Net-(U2-GND-Pad29) -> GND
- U2 pad 3: Net-(U2-GND-Pad29) -> GND
- U2 pad 4: unconnected-(U2-D+-Pad4) -> /D+
- U2 pad 5: unconnected-(U2-D--Pad5) -> /D-
- U2 pad 6: unconnected-(U2-VDD-Pad6) -> /V3.3
- U2 pad 7: unconnected-(U2-REGIN-Pad7) -> /V3.3
- U2 pad 8: unconnected-(U2-VBUS-Pad8) -> /VBUS
- U2 pad 9: unconnected-(U2-~{RST}-Pad9) -> Net-(U2-~{RST})
Routing:
- net /V3.3: track 0.00 -> 281.9 mm, vias 0 -> 15
- net /VOUT: track 0.00 -> 207.4 mm, vias 0 -> 8
- net GND: track 0.00 -> 154.2 mm, vias 0 -> 25
- net /VBUS: track 0.00 -> 97.1 mm, vias 0 -> 6
- net /SCL: track 0.00 -> 89.1 mm, vias 0 -> 2
- net /S_touch_5: track 0.00 -> 81.6 mm, vias 0 -> 1
- net /SDA: track 0.00 -> 80.8 mm, vias 0 -> 4
- net /TX0: track 0.00 -> 79.4 mm, vias 0 -> 2
- net /RX0: track 0.00 -> 74.8 mm, vias 0 -> 2
- net /IO7: track 0.00 -> 70.5 mm, vias 0 -> 2
- net /IO6: track 0.00 -> 70.5 mm, vias 0 -> 2
- net /IO4: track 0.00 -> 70.4 mm, vias 0 -> 2
- net /IO5: track 0.00 -> 70.3 mm, vias 0 -> 2
- net /S_touch_2: track 0.00 -> 69.4 mm, vias 0 -> 1
- net /S_touch_4: track 0.00 -> 67.4 mm, vias 0 -> 1
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- added copper zone on B.Cu, net GND
- added copper zone on F.Cu, net GND
Other:
- board outline added: 150 x 100 mm
- copper layers 2 -> 4
- board text added: "BATTERY"

Commit message: Initialize first pcb version
Parts:
- removed U2: CP2102, CP2102:QFN50P500X500X100-29N
- added REF**: MountingHole_2.7mm_M2.5_DIN965_Pad, MountingHole:MountingHole_2.7mm_M2.5_DIN965_Pad, F.Cu at (42.0, 63.0)
- added REF**: MountingHole_2.7mm_M2.5_DIN965_Pad, MountingHole:MountingHole_2.7mm_M2.5_DIN965_Pad, F.Cu at (42.0, 39.0)
- added REF**: MountingHole_2.7mm_M2.5_Pad_Via, MountingHole:MountingHole_2.7mm_M2.5_Pad_Via, F.Cu at (8.00, 8.00)
- added REF**: MountingHole_2.7mm_M2.5_Pad_Via, MountingHole:MountingHole_2.7mm_M2.5_Pad_Via, F.Cu at (8.00, 92.0)
- added REF**: MountingHole_2.7mm_M2.5_Pad_Via, MountingHole:MountingHole_2.7mm_M2.5_Pad_Via, F.Cu at (142.0, 92.0)
- added REF**: MountingHole_2.7mm_M2.5_DIN965_Pad, MountingHole:MountingHole_2.7mm_M2.5_DIN965_Pad, F.Cu at (18.0, 63.0)
- added REF**: MountingHole_2.7mm_M2.5_DIN965_Pad, MountingHole:MountingHole_2.7mm_M2.5_DIN965_Pad, F.Cu at (18.0, 39.0)
- added REF**: MountingHole_2.7mm_M2.5_Pad_Via, MountingHole:MountingHole_2.7mm_M2.5_Pad_Via, F.Cu at (142.0, 8.00)
- added U6: CP2102, CP2102:QFN50P500X500X100-29N, B.Cu at (123.1, 9.32)
- moved BT1 16.6 mm to (128.5, 90.0)
- renumbered D8 to RGB
Routing:
- net GND: track 154.2 -> 178.5 mm, vias 25 -> 29
- net /BAT: track 51.7 -> 67.8 mm
- net /V3.3: track 281.9 -> 292.1 mm
- net /IO5: track 70.3 -> 69.1 mm
- net /IO4: track 70.4 -> 69.2 mm
- net /IO6: track 70.5 -> 69.4 mm
- net /IO7: track 70.5 -> 69.5 mm
- net /LCD_RESET: track 58.6 -> 57.9 mm
- net /LCD_WR: track 51.7 -> 51.0 mm
- net /LCD_RS/DC: track 51.0 -> 50.4 mm
Other:
- outline, holes or cut-outs redrawn
- copper layers 4 -> 2
- board text added: "Designed by kokh.me"
- board text added: "Smart Core Demo"
- board text added: "V1"
